Commit message: add ros_ship_gazebo_plugins package

File: ros_ship_description/robots/ros_ship.urdf.xacro (robot description, xacro)
@@ -6,4 +6,6 @@
   <xacro:property name="motor_position_y" value="0.325" />
   <xacro:property name="motor_position_z" value="-0.15" />
+  <xacro:property name="cob" value="0.0 0.0 -0.3"/>
+  <xacro:property name="volume" value="30000"/>
   <link name="base_footprint"/>
   <joint name="base_link_joint" type="fixed">
@@ -24,8 +26,9 @@
     </collision>
     <inertial>
-      <mass value="95.7802"/>
+      <mass value="95.78"/>
       <inertia ixx="57.28" ixy="0.00" ixz="-0.23" iyy="57.28" iyz="0.00" izz="6.09"/>
     </inertial>
   </link>
+<!--
   <xacro:include filename="$(find velodyne_description)/urdf/VLP-16.urdf.xacro"/>
   <VLP-16 parent="base_link" name="velodyne" topic="/velodyne_points">
@@ -199,7 +202,4 @@
         <noise>
           <type>gaussian</type>
-          <!-- Noise is sampled independently per pixel on each frame.
-               That pixel's noise value is added to each of its color
-               channels, which at that point lie in the range [0,1]. -->
           <mean>0.0</mean>
           <stddev>0.007</stddev>
@@ -238,7 +238,4 @@
         <noise>
           <type>gaussian</type>
-          <!-- Noise is sampled independently per pixel on each frame.
-               That pixel's noise value is added to each of its color
-               channels, which at that point lie in the range [0,1]. -->
           <mean>0.0</mean>
           <stddev>0.007</stddev>
@@ -261,3 +258,19 @@
     </sensor>
   </gazebo>
+-->
+  <gazebo>
+    <plugin name="simple_buoyancy" filename="libsimple_buoyancy_plugin.so">
+      <target_link>base_footprint</target_link>
+      <water_surface_height>1</water_surface_height>
+      <cob_x>0.375</cob_x>
+      <cob_y>0</cob_y>
+      <cob_z>0.25</cob_z>
+      <bbox_x>2.75</bbox_x>
+      <bbox_y>1.0</bbox_y>
+      <bbox_z>0.5</bbox_z>
+    </plugin>
+    <plugin name="simple_buoyancy" filename="libworld_frame_publisher_plugin.so">
+      <reference_link>base_footprint</reference_link>
+    </plugin>
+  </gazebo>
 </robot>

File: ros_ship_description/urdf/ros_ship.urdf (robot description, URDF)
Before this commit: robot ros_ship, 9 links, 8 joints
Links:
- added link velodyne_base_link, mass 0.1; collision cylinder length=0.0717 radius=0.0516; visual mesh filename=package://velodyne_description/meshes/VLP16_base_1.dae
- link camera_l: mass None -> 0.01
- link camera_r: mass None -> 0.01
- link motor_l: mass None -> 0.28
- link motor_r: mass None -> 0.28
- link propeller_l: mass None -> 0.28
- link propeller_r: mass None -> 0.28
- link velodyne: mass None -> 0.1; geometry visual mesh filename=package://velodyne_description/meshes/VLP16_scan.dae
Joints:
- removed joint velodyne_joint
- added joint velodyne_base_mount_joint: type fixed, parent base_link, child velodyne_base_link, origin xyz=1.4 0 0.55 rpy=0 0 0
- added joint velodyne_base_scan_joint: type fixed, parent velodyne_base_link, child velodyne, origin xyz=0 0 0.0377 rpy=0 0 0
- joint propeller_l_joint: origin xyz=0.17 0 0.026 -> xyz=0.17 0 0.026 rpy=0 0 3.14159265359
- joint propeller_r_joint: origin xyz=0.17 0 0.026 -> xyz=0.17 0 0.026 rpy=0 0 3.14159265359

Commit message: add WATER_SURFACE.world

File: ros_ship_description/robots/ros_ship.urdf.xacro (robot description, xacro)
@@ -30,5 +30,4 @@
     </inertial>
   </link>
-<!--
   <xacro:include filename="$(find velodyne_description)/urdf/VLP-16.urdf.xacro"/>
   <VLP-16 parent="base_link" name="velodyne" topic="/velodyne_points">
@@ -52,5 +51,5 @@
     </collision>
     <inertial>
-      <mass value="0.01"/>
+      <mass value="0.0"/>
       <inertia ixx="0.00" ixy="0.00" ixz="0.00" iyy="0.00" iyz="0.00" izz="0.00"/>
     </inertial>
@@ -73,5 +72,5 @@
     </collision>
     <inertial>
-      <mass value="0.01"/>
+      <mass value="0.0"/>
       <inertia ixx="0.00" ixy="0.00" ixz="0.00" iyy="0.00" iyz="0.00" izz="0.00"/>
     </inertial>
@@ -94,5 +93,5 @@
     </collision>
     <inertial>
-      <mass value="0.28"/>
+      <mass value="0.0001"/>
       <inertia ixx="0.0001" ixy="0.00" ixz="0.00" iyy="0.0001" iyz="0.00" izz="0.0001"/>
     </inertial>
@@ -115,5 +114,5 @@
     </collision>
     <inertial>
-      <mass value="0.28"/>
+      <mass value="0.0001"/>
       <inertia ixx="0.00086" ixy="0.00" ixz="0.00" iyy="0.00086" iyz="0.00" izz="0.0017"/>
     </inertial>
@@ -136,5 +135,5 @@
     </collision>
     <inertial>
-      <mass value="0.28"/>
+      <mass value="0.0001"/>
       <inertia ixx="0.00" ixy="0.00" ixz="0.00" iyy="0.00" iyz="0.00" izz="0.00"/>
     </inertial>
@@ -157,5 +156,5 @@
     </collision>
     <inertial>
-      <mass value="0.28"/>
+      <mass value="0.0001"/>
       <inertia ixx="0.00086" ixy="0.00" ixz="0.00" iyy="0.00086" iyz="0.00" izz="0.0017"/>
     </inertial>
@@ -258,5 +257,4 @@
     </sensor>
   </gazebo>
--->
   <gazebo>
     <plugin name="simple_buoyancy" filename="libsimple_buoyancy_plugin.so">
@@ -270,4 +268,24 @@
       <publish_data>true</publish_data>
     </plugin>
+    <plugin name="simple_buoyancy" filename="libsimple_buoyancy_plugin.so">
+      <target_link>propeller_r</target_link>
+      <cob_x>0.1</cob_x>
+      <cob_y>0.0</cob_y>
+      <cob_z>0.0</cob_z>
+      <bbox_x>0.1</bbox_x>
+      <bbox_y>0.2</bbox_y>
+      <bbox_z>0.2</bbox_z>
+      <publish_data>true</publish_data>
+    </plugin>
+    <plugin name="simple_buoyancy" filename="libsimple_buoyancy_plugin.so">
+      <target_link>propeller_l</target_link>
+      <cob_x>0.1</cob_x>
+      <cob_y>0.0</cob_y>
+      <cob_z>0.0</cob_z>
+      <bbox_x>0.1</bbox_x>
+      <bbox_y>0.2</bbox_y>
+      <bbox_z>0.2</bbox_z>
+      <publish_data>true</publish_data>
+    </plugin>
     <plugin name="simple_buoyancy" filename="libworld_frame_publisher_plugin.so">
       <reference_link>base_footprint</reference_link>

Commit message: add right and left motor

File: ros_ship_description/robots/ros_ship.urdf.xacro (robot description, xacro)
@@ -114,5 +114,5 @@
     </collision>
     <inertial>
-      <mass value="0.0001"/>
+      <mass value="0.001"/>
       <inertia ixx="0.00086" ixy="0.00" ixz="0.00" iyy="0.00086" iyz="0.00" izz="0.0017"/>
     </inertial>
@@ -165,5 +165,5 @@
       <hardwareInterface>VelocityJointInterface</hardwareInterface>
     </joint>
-    <actuator name="motor_r_actuator">
+    <actuator name="right_motor_actuator">
       <hardwareInterface>VelocityJointInterface</hardwareInterface>
       <mechanicalReduction>30</mechanicalReduction>

File: ros_ship_description/urdf/ros_ship.urdf (robot description, URDF)
Before this commit: robot ros_ship, 10 links, 9 joints
Links:
- link base_link: mass 95.7802 -> 95.78
- link camera_l: mass 0.01 -> 0.0
- link camera_r: mass 0.01 -> 0.0
- link motor_l: mass 0.28 -> 0.0001
- link motor_r: mass 0.28 -> 0.0001
- link propeller_l: mass 0.28 -> 0.0001
- link propeller_r: mass 0.28 -> 0.0001
