Commit message: add simple_driving_force_plugin

File: ros_ship_description/robots/wam-v.urdf.xacro (robot description, xacro)
@@ -12,4 +12,6 @@
   <xacro:property name="motor_size_y" value="0.2" />
   <xacro:property name="motor_size_z" value="0.2" />
+  <xacro:property name="rotational_speed_effort" value="1" />
+  <xacro:property name="joint_state_topic" value="/wam_v/joint_states" />
   <link name="base_link">
     <visual>
@@ -76,4 +78,10 @@
     <child link="left_motor"/>
   </joint>
+  <link name="gps"/>
+  <joint name="gps_joint" type="fixed">
+    <origin xyz="0.8 0 0"/>
+    <parent link="base_link"/>
+    <child link="gps"/>
+  </joint>
   <transmission name="right_motor_trans">
     <type>transmission_interface/SimpleTransmission</type>
@@ -100,5 +108,5 @@
       <robotNamespace>/wam_v</robotNamespace>
     </plugin>
-    <plugin name="simple_buoyancy" filename="libsimple_buoyancy_plugin.so">
+    <plugin name="simple_buoyancy_base_right" filename="libsimple_buoyancy_plugin.so">
       <target_link>base_link</target_link>
       <cob_x>${hal_position_x}</cob_x>
@@ -111,5 +119,5 @@
       <bbox_prefix>right_bbox</bbox_prefix>
     </plugin>
-    <plugin name="simple_buoyancy" filename="libsimple_buoyancy_plugin.so">
+    <plugin name="simple_buoyancy_base_left" filename="libsimple_buoyancy_plugin.so">
       <target_link>base_link</target_link>
       <cob_x>${hal_position_x}</cob_x>
@@ -122,5 +130,5 @@
       <bbox_prefix>left_bbox</bbox_prefix>
     </plugin>
-    <plugin name="simple_buoyancy" filename="libsimple_buoyancy_plugin.so">
+    <plugin name="simple_buoyancy_motor_right" filename="libsimple_buoyancy_plugin.so">
       <target_link>right_motor</target_link>
       <cob_x>0</cob_x>
@@ -132,5 +140,5 @@
       <publish_data>true</publish_data>
     </plugin>
-    <plugin name="simple_buoyancy" filename="libsimple_buoyancy_plugin.so">
+    <plugin name="simple_buoyancy_motor_left" filename="libsimple_buoyancy_plugin.so">
       <target_link>left_motor</target_link>
       <cob_x>0</cob_x>
@@ -142,4 +150,29 @@
       <publish_data>true</publish_data>
     </plugin>
+    <plugin name="novatel_gps_sim" filename="libhector_gazebo_ros_gps.so">
+      <alwaysOn>1</alwaysOn>
+      <updateRate>10.0</updateRate>
+      <bodyName>gps</bodyName>
+      <topicName>fix</topicName>
+      <velocityTopicName>fix_velocity</velocityTopicName>
+      <drift>5.0 5.0 5.0</drift>
+      <gaussianNoise>0.1 0.1 0.1</gaussianNoise>
+      <velocityDrift>0 0 0</velocityDrift>
+      <velocityGaussianNoise>0.1 0.1 0.1</velocityGaussianNoise>
+    </plugin>
+  </gazebo>
+  <gazebo>
+    <plugin name="simple_driving_force_left" filename="libsimple_driving_force_plugin.so">
+      <target_link>left_motor</target_link>
+      <target_joint>left_motor_joint</target_joint>
+      <rotational_speed_effort>${rotational_speed_effort}</rotational_speed_effort>
+      <joint_state_topic>${joint_state_topic}</joint_state_topic>
+    </plugin>
+    <plugin name="simple_driving_force_right" filename="libsimple_driving_force_plugin.so">
+      <target_link>right_motor</target_link>
+      <target_joint>right_motor_joint</target_joint>
+      <rotational_speed_effort>${rotational_speed_effort}</rotational_speed_effort>
+      <joint_state_topic>${joint_state_topic}</joint_state_topic>
+    </plugin>
   </gazebo>
 </robot>

Commit message: add robot_pose_ekf node and odom frame

File: ros_ship_description/robots/wam-v.urdf.xacro (robot description, xacro)
@@ -2,5 +2,5 @@
   <xacro:property name="hal_position_x" value="0.5" />
   <xacro:property name="hal_position_y" value="1.05" />
-  <xacro:property name="hal_position_z" value="-1.25" />
+  <xacro:property name="hal_position_z" value="0.5" />
   <xacro:property name="hal_size_x" value="4.0" />
   <xacro:property name="hal_size_y" value="0.5" />
@@ -30,8 +30,8 @@
    </inertial>
   </link>
-  <joint name="base_footprint_joint" type="fixed">
-    <origin xyz="0 0 -1.84"/>
-    <parent link="base_link"/>
-    <child link="base_footprint"/>
+  <joint name="base_link_joint" type="fixed">
+    <origin xyz="0 0 1.84"/>
+    <parent link="base_footprint"/>
+    <child link="base_link"/>
   </joint>
   <link name="base_footprint"/>
@@ -109,5 +109,5 @@
     </plugin>
     <plugin name="simple_buoyancy_base_right" filename="libsimple_buoyancy_plugin.so">
-      <target_link>base_link</target_link>
+      <target_link>base_footprint</target_link>
       <cob_x>${hal_position_x}</cob_x>
       <cob_y>-${hal_position_y}</cob_y>
@@ -120,5 +120,5 @@
     </plugin>
     <plugin name="simple_buoyancy_base_left" filename="libsimple_buoyancy_plugin.so">
-      <target_link>base_link</target_link>
+      <target_link>base_footprint</target_link>
       <cob_x>${hal_position_x}</cob_x>
       <cob_y>${hal_position_y}</cob_y>
@@ -152,5 +152,5 @@
     <plugin name="novatel_gps_sim" filename="libhector_gazebo_ros_gps.so">
       <alwaysOn>1</alwaysOn>
-      <updateRate>10.0</updateRate>
+      <updateRate>10</updateRate>
       <bodyName>gps</bodyName>
       <topicName>fix</topicName>
@@ -161,6 +161,4 @@
       <velocityGaussianNoise>0.1 0.1 0.1</velocityGaussianNoise>
     </plugin>
-  </gazebo>
-  <gazebo>
     <plugin name="simple_driving_force_left" filename="libsimple_driving_force_plugin.so">
       <target_link>left_motor</target_link>
@@ -175,9 +173,12 @@
       <joint_state_topic>${joint_state_topic}</joint_state_topic>
     </plugin>
-    <!--
-    <plugin name="simple_driving_force_right" filename="libworld_frame_publisher_plugin.so">
-      <reference_link>base_link</reference_link>
+    <plugin name="imu_plugin" filename="libgazebo_ros_imu.so">
+      <alwaysOn>true</alwaysOn>
+      <bodyName>base_link</bodyName>
+      <topicName>imu</topicName>
+      <serviceName>imu_service</serviceName>
+      <gaussianNoise>0.0</gaussianNoise>
+      <updateRate>20.0</updateRate>
     </plugin>
-    -->
   </gazebo>
 </robot>

Commit message: add joy_to_cmd node

File: ros_ship_description/robots/wam-v.urdf.xacro (robot description, xacro)
@@ -56,4 +56,5 @@
     <parent link="base_link"/>
     <child link="right_motor"/>
+    <limit effort="0.5293" velocity="100${pi}" />
   </joint>
   <link name="left_motor">
@@ -77,4 +78,5 @@
     <parent link="base_link"/>
     <child link="left_motor"/>
+    <limit effort="0.5293" velocity="100${pi}" />
   </joint>
   <link name="gps"/>
@@ -132,7 +134,8 @@
     <plugin name="simple_buoyancy_motor_right" filename="libsimple_buoyancy_plugin.so">
       <target_link>right_motor</target_link>
-      <cob_x>0</cob_x>
-      <cob_y>0</cob_y>
-      <cob_z>0.5</cob_z>
+      <position_reference_link>base_footprint</position_reference_link>
+      <cob_x>-1.5</cob_x>
+      <cob_y>-1</cob_y>
+      <cob_z>0.3</cob_z>
       <bbox_x>${motor_size_x}</bbox_x>
       <bbox_y>${motor_size_y}</bbox_y>
@@ -142,7 +145,8 @@
     <plugin name="simple_buoyancy_motor_left" filename="libsimple_buoyancy_plugin.so">
       <target_link>left_motor</target_link>
-      <cob_x>0</cob_x>
-      <cob_y>0</cob_y>
-      <cob_z>0.5</cob_z>
+      <position_reference_link>base_footprint</position_reference_link>
+      <cob_x>-1.5</cob_x>
+      <cob_y>1</cob_y>
+      <cob_z>0.3</cob_z>
       <bbox_x>${motor_size_x}</bbox_x>
       <bbox_y>${motor_size_y}</bbox_y>

Commit message: modify axes index

File: ros_ship_description/robots/wam-v.urdf.xacro (robot description, xacro)
@@ -10,6 +10,6 @@
   <xacro:property name="motor_position_z" value="-1.705" />
   <xacro:property name="motor_size_x" value="0.1" />
-  <xacro:property name="motor_size_y" value="0.2" />
-  <xacro:property name="motor_size_z" value="0.2" />
+  <xacro:property name="motor_size_y" value="0.5" />
+  <xacro:property name="motor_size_z" value="0.5" />
   <xacro:property name="rotational_speed_effort" value="1" />
   <xacro:property name="joint_state_topic" value="/wam_v/joint_states" />
@@ -137,5 +137,5 @@
       <cob_x>-1.5</cob_x>
       <cob_y>-1</cob_y>
-      <cob_z>0.3</cob_z>
+      <cob_z>0.5</cob_z>
       <bbox_x>${motor_size_x}</bbox_x>
       <bbox_y>${motor_size_y}</bbox_y>
@@ -148,5 +148,5 @@
       <cob_x>-1.5</cob_x>
       <cob_y>1</cob_y>
-      <cob_z>0.3</cob_z>
+      <cob_z>0.5</cob_z>
       <bbox_x>${motor_size_x}</bbox_x>
       <bbox_y>${motor_size_y}</bbox_y>

Commit message: add force_offcet_x,y,z value

File: ros_ship_description/robots/wam-v.urdf.xacro (robot description, xacro)
@@ -10,6 +10,6 @@
   <xacro:property name="motor_position_z" value="-1.705" />
   <xacro:property name="motor_size_x" value="0.1" />
-  <xacro:property name="motor_size_y" value="0.5" />
-  <xacro:property name="motor_size_z" value="0.5" />
+  <xacro:property name="motor_size_y" value="0.2" />
+  <xacro:property name="motor_size_z" value="0.2" />
   <xacro:property name="rotational_speed_effort" value="1" />
   <xacro:property name="joint_state_topic" value="/wam_v/joint_states" />
@@ -120,4 +120,5 @@
       <publish_data>true</publish_data>
       <bbox_prefix>right_bbox</bbox_prefix>
+      <force_offset_x>0.01</force_offset_x>
     </plugin>
     <plugin name="simple_buoyancy_base_left" filename="libsimple_buoyancy_plugin.so">
@@ -131,4 +132,5 @@
       <publish_data>true</publish_data>
       <bbox_prefix>left_bbox</bbox_prefix>
+      <force_offset_x>0.01</force_offset_x>
     </plugin>
     <plugin name="simple_buoyancy_motor_right" filename="libsimple_buoyancy_plugin.so">
@@ -137,5 +139,5 @@
       <cob_x>-1.5</cob_x>
       <cob_y>-1</cob_y>
-      <cob_z>0.5</cob_z>
+      <cob_z>0.2</cob_z>
       <bbox_x>${motor_size_x}</bbox_x>
       <bbox_y>${motor_size_y}</bbox_y>
@@ -148,5 +150,5 @@
       <cob_x>-1.5</cob_x>
       <cob_y>1</cob_y>
-      <cob_z>0.5</cob_z>
+      <cob_z>0.2</cob_z>
       <bbox_x>${motor_size_x}</bbox_x>
       <bbox_y>${motor_size_y}</bbox_y>

Commit message: add ros_ship_visualization package

File: ros_ship_description/robots/wam-v.urdf.xacro (robot description, xacro)
@@ -14,4 +14,6 @@
   <xacro:property name="rotational_speed_effort" value="1" />
   <xacro:property name="joint_state_topic" value="/wam_v/joint_states" />
+  <xacro:property name="start_point_latitude" value="135.525" />
+  <xacro:property name="start_point_longitude" value="34.8235" />
   <link name="base_link">
     <visual>
@@ -168,4 +170,6 @@
       <velocityDrift>0 0 0</velocityDrift>
       <velocityGaussianNoise>0.1 0.1 0.1</velocityGaussianNoise>
+      <referenceLatitude>${start_point_latitude}</referenceLatitude>
+      <referenceLongitude>${start_point_longitude}</referenceLongitude>
     </plugin>
     <plugin name="simple_driving_force_left" filename="libsimple_driving_force_plugin.so">

Commit message: add camera and lrf

File: ros_ship_description/robots/wam-v.urdf.xacro (robot description, xacro)
@@ -1,19 +1,5 @@
+<?xml version="1.0"?>
 <robot xmlns:xacro="http://ros.org/wiki/xacro" name="wam-v">
-  <xacro:property name="hal_position_x" value="0.5" />
-  <xacro:property name="hal_position_y" value="1.05" />
-  <xacro:property name="hal_position_z" value="0.5" />
-  <xacro:property name="hal_size_x" value="4.0" />
-  <xacro:property name="hal_size_y" value="0.5" />
-  <xacro:property name="hal_size_z" value="0.5" />
-  <xacro:property name="motor_position_x" value="-1.5" />
-  <xacro:property name="motor_position_y" value="1.027" />
-  <xacro:property name="motor_position_z" value="-1.705" />
-  <xacro:property name="motor_size_x" value="0.1" />
-  <xacro:property name="motor_size_y" value="0.2" />
-  <xacro:property name="motor_size_z" value="0.2" />
-  <xacro:property name="rotational_speed_effort" value="1" />
-  <xacro:property name="joint_state_topic" value="/wam_v/joint_states" />
-  <xacro:property name="start_point_latitude" value="135.525" />
-  <xacro:property name="start_point_longitude" value="34.8235" />
+  <xacro:include filename="properties.urdf.xacro"/>
   <link name="base_link">
     <visual>
@@ -38,4 +24,28 @@
   </joint>
   <link name="base_footprint"/>
+  <link name="front_camera_link"/>
+  <joint name="front_camera_joint" type="fixed">
+    <origin xyz="1.2 0 0"/>
+    <parent link="base_link"/>
+    <child link="front_camera_link"/>
+  </joint>
+  <link name="left_camera_link"/>
+  <joint name="left_camera_joint" type="fixed">
+    <origin xyz="0 0.5 0" rpy="0 0 ${pi/2}"/>
+    <parent link="base_link"/>
+    <child link="left_camera_link"/>
+  </joint>
+  <link name="right_camera_link"/>
+  <joint name="right_camera_joint" type="fixed">
+    <origin xyz="0 -0.5 0" rpy="0 0 ${-pi/2}"/>
+    <parent link="base_link"/>
+    <child link="right_camera_link"/>
+  </joint>
+  <link name="rear_camera_link"/>
+  <joint name="rear_camera_joint" type="fixed">
+    <origin xyz="-0.5 0 0" rpy="0 0 ${pi}"/>
+    <parent link="base_link"/>
+    <child link="rear_camera_link"/>
+  </joint>
   <link name="right_motor">
     <visual>
@@ -110,5 +120,5 @@
   <gazebo>
     <plugin name="gazebo_ros_control" filename="libgazebo_ros_control.so">
-      <robotNamespace>/wam_v</robotNamespace>
+      <robotNamespace>${robot}</robotNamespace>
     </plugin>
     <plugin name="simple_buoyancy_base_right" filename="libsimple_buoyancy_plugin.so">
@@ -176,5 +186,5 @@
       <target_link>left_motor</target_link>
       <target_joint>left_motor_joint</target_joint>
-      <driving_force_controller>/wam_v/right_driving_force_controller</driving_force_controller>
+      <driving_force_controller>/${robot}/right_driving_force_controller</driving_force_controller>
       <joint_state_topic>${joint_state_topic}</joint_state_topic>
     </plugin>
@@ -182,5 +192,5 @@
       <target_link>right_motor</target_link>
       <target_joint>right_motor_joint</target_joint>
-      <driving_force_controller>/wam_v/left_driving_force_controller</driving_force_controller>
+      <driving_force_controller>/${robot}/left_driving_force_controller</driving_force_controller>
       <joint_state_topic>${joint_state_topic}</joint_state_topic>
     </plugin>
@@ -199,3 +209,12 @@
     </plugin>
   </gazebo>
+  <xacro:include filename="camera.urdf.xacro"/>
+  <xacro:camera prefix="front"/>
+  <xacro:camera prefix="right"/>
+  <xacro:camera prefix="left"/>
+  <xacro:camera prefix="rear"/>
+  <xacro:include filename="$(find velodyne_description)/urdf/VLP-16.urdf.xacro"/>
+  <VLP-16 parent="base_link" name="velodyne" topic="/velodyne_points">
+    <origin xyz="0.9 0 0.3" rpy="0 0 0" />
+  </VLP-16>
 </robot>

Commit message: add laser sensor

File: ros_ship_description/robots/wam-v.urdf.xacro (robot description, xacro)
@@ -15,5 +15,5 @@
    <inertial>
      <mass value="247.07"/>
-     <inertia ixx="200" ixy="0.03" ixz="3.09" iyy="181.69" iyz="-0.05" izz="165.39"/>
+     <inertia ixx="200" ixy="0.03" ixz="3.09" iyy="500" iyz="-0.05" izz="165.39"/>
    </inertial>
   </link>
@@ -47,4 +47,10 @@
     <parent link="base_link"/>
     <child link="rear_camera_link"/>
+  </joint>
+  <link name="scan"/>
+  <joint name="scan_joint" type="fixed">
+    <origin xyz="1.5 0 -1" rpy="0 0 0"/>
+    <parent link="base_link"/>
+    <child link="scan"/>
   </joint>
   <link name="right_motor">
@@ -216,5 +222,33 @@
   <xacro:include filename="$(find velodyne_description)/urdf/VLP-16.urdf.xacro"/>
   <VLP-16 parent="base_link" name="velodyne" topic="/velodyne_points">
-    <origin xyz="0.9 0 0.3" rpy="0 0 0" />
+    <origin xyz="0.8 0 0.3" rpy="0 0 0" />
   </VLP-16>
+  <gazebo reference="scan">
+    <material>Gazebo/Blue</material>
+    <turnGravityOff>false</turnGravityOff>
+    <sensor type="ray" name="scan_sensor">
+      <pose>0 0 0 0 0 0</pose>
+      <visualize>false</visualize>
+      <update_rate>40</update_rate>
+      <ray>
+        <scan>
+          <horizontal>
+            <samples>720</samples>
+            <resolution>1</resolution>
+            <min_angle>-1.570796</min_angle>
+            <max_angle>1.570796</max_angle>
+          </horizontal>
+        </scan>
+        <range>
+          <min>1</min>
+          <max>30.0</max>
+          <resolution>0.001</resolution>
+        </range>
+      </ray>
+      <plugin name="gazebo_ros_head_hokuyo_controller" filename="libgazebo_ros_laser.so">
+        <topicName>/scan</topicName>
+        <frameName>scan</frameName>
+      </plugin>
+    </sensor>
+  </gazebo>
 </robot>
