Commit message: add kml_plotter node

File: ros_ship_description/robots/properties.urdf.xacro (robot description, xacro)
@@ -15,6 +15,6 @@
   <xacro:property name="rotational_speed_effort" value="1" />
   <xacro:property name="joint_state_topic" value="/wam_v/joint_states" />
-  <xacro:property name="start_point_latitude" value="135.525" />
-  <xacro:property name="start_point_longitude" value="34.8235" />
+  <xacro:property name="start_point_latitude" value="135.524910" />
+  <xacro:property name="start_point_longitude" value="34.822634" />
   <xacro:property name="robot" value="wam_v" />
 </robot>

Commit message: remove twist_topic parameters from simple_driving_force plugin

File: ros_ship_description/robots/properties.urdf.xacro (robot description, xacro)
@@ -17,4 +17,5 @@
   <xacro:property name="start_point_latitude" value="135.524910" />
   <xacro:property name="start_point_longitude" value="34.822634" />
+  <xacro:property name="start_point_heading" value="0" />
   <xacro:property name="robot" value="wam_v" />
 </robot>

File: ros_ship_description/robots/wam-v.urdf.xacro (robot description, xacro)
@@ -188,4 +188,5 @@
       <referenceLatitude>${start_point_latitude}</referenceLatitude>
       <referenceLongitude>${start_point_longitude}</referenceLongitude>
+      <referenceHeading>${start_point_heading}</referenceHeading>
     </plugin>
     <plugin name="simple_driving_force_left" filename="libsimple_driving_force_plugin.so">

File: ros_ship_description/urdf/wam-v.urdf (robot description, URDF)
Before this commit: robot wam-v, 4 links, 2 joints
Links:
- added link front_camera_link
- added link gps
- added link left_camera_link
- added link rear_camera_link
- added link right_camera_link
- added link scan
- added link velodyne, mass 0.1; visual mesh filename=package://velodyne_description/meshes/VLP16_scan.dae
- added link velodyne_base_link, mass 0.1; collision cylinder length=0.0717 radius=0.0516; visual mesh filename=package://velodyne_description/meshes/VLP16_base_1.dae
- link left_motor: mass 0.0001 -> 0.01
- link right_motor: mass 0.0001 -> 0.01
Joints:
- removed joint base_footprint_joint
- added joint base_link_joint: type fixed, parent base_footprint, child base_link, origin xyz=0 0 1.84
- added joint front_camera_joint: type fixed, parent base_link, child front_camera_link, origin xyz=1.2 0 0
- added joint gps_joint: type fixed, parent base_link, child gps, origin xyz=0.8 0 0
- added joint left_camera_joint: type fixed, parent base_link, child left_camera_link, origin xyz=0 0.5 0 rpy=0 0 1.57079632679
- added joint rear_camera_joint: type fixed, parent base_link, child rear_camera_link, origin xyz=-0.5 0 0 rpy=0 0 3.14159265359
- added joint right_camera_joint: type fixed, parent base_link, child right_camera_link, origin xyz=0 -0.5 0 rpy=0 0 -1.57079632679
- added joint right_motor_joint: type continuous, parent base_link, child right_motor, origin xyz=-1.5 -1.027 -1.705, limit effort=0.5293 velocity=1003.14159265359
- added joint scan_joint: type fixed, parent base_link, child scan, origin xyz=1.5 0 -1 rpy=0 0 0
- added joint velodyne_base_mount_joint: type fixed, parent base_link, child velodyne_base_link, origin xyz=0.8 0 0.3 rpy=0 0 0
- added joint velodyne_base_scan_joint: type fixed, parent velodyne_base_link, child velodyne, origin xyz=0 0 0.0377 rpy=0 0 0
- joint left_motor_joint: limit (none) -> effort=0.5293 velocity=1003.14159265359; origin xyz=-0.5 0.75 -1.5 -> xyz=-1.5 1.027 -1.705
